File: AXK770147G_breakout/AXK770147G_breakout.sch (KiCad schematic (older format))
At the start: 4 parts, among them J1 Conn_01x35, J2 Conn_01x18, J3 AXK770147G, J4 Conn_01x17

Commit message: Move traces around a bit to increase separation; add ground pins.
Parts:
- J1: value Conn_01x35 -> Conn_01x36; symbol Connector_Generic:Conn_01x35 -> Connector_Generic:Conn_01x36
- J4: value Conn_01x17 -> Conn_01x18; footprint Connector_PinHeader_2.54mm:PinHeader_1x17_P2.54mm_Vertical -> Connector_PinHeader_2.54mm:PinHeader_1x18_P2.54mm_Vertical; symbol Connector_Generic:Conn_01x17 -> Connector_Generic:Conn_01x18
Connections:
- net at J3.37: now also J4.2 (Pin_2); no longer J4.1 (Pin_1)
- net at J3.39: now also J4.3 (Pin_3); no longer J4.2 (Pin_2)
- net at J3.41: now also J4.4 (Pin_4); no longer J4.3 (Pin_3)
- net at J3.43: now also J4.5 (Pin_5); no longer J4.4 (Pin_4)
- net at J3.45: now also J4.6 (Pin_6); no longer J4.5 (Pin_5)
- net at J3.47: now also J4.7 (Pin_7); no longer J4.6 (Pin_6)
- net at J3.49: now also J4.8 (Pin_8); no longer J4.7 (Pin_7)
- net at J3.51: now also J4.9 (Pin_9); no longer J4.8 (Pin_8)
- net at J3.53: now also J4.10 (Pin_10); no longer J4.9 (Pin_9)
- net at J3.55: now also J4.11 (Pin_11); no longer J4.10 (Pin_10)
- net at J3.57: now also J4.12 (Pin_12); no longer J4.11 (Pin_11)
- net at J3.59: now also J4.13 (Pin_13); no longer J4.12 (Pin_12)
- net at J3.61: now also J4.14 (Pin_14); no longer J4.13 (Pin_13)
- net at J3.63: now also J4.15 (Pin_15); no longer J4.14 (Pin_14)
- net at J3.65: now also J4.16 (Pin_16); no longer J4.15 (Pin_15)
- net at J3.67: now also J4.17 (Pin_17); no longer J4.16 (Pin_16)
- net at J3.69: now also J4.18 (Pin_18); no longer J4.17 (Pin_17)
- new net GND: J1.36 (Pin_36), J4.1 (Pin_1)
Changed lines of the file:
@@
 $EndComp
 $Comp
-L Connector_Generic:Conn_01x35 J1
+L Connector_Generic:Conn_01x36 J1
 U 1 1 601EB970
 P 5750 600
 F 0 "J1" V 5967 596 50  0000 C CNN
-F 1 "Conn_01x35" V 5876 596 50  0000 C CNN
+F 1 "Conn_01x36" V 5876 596 50  0000 C CNN
 F 2 "Connector_PinHeader_2.54mm:PinHeader_2x18_P2.54mm_Vertical" H 5750 600 50  0001 C CNN
 F 3 "~" H 5750 600 50  0001 C CNN
@@
 	8600 4950 8600 6250
 $Comp
-L Connector_Generic:Conn_01x17 J4
+L Connector_Generic:Conn_01x18 J4
 U 1 1 60503150
-P 4850 6400
-F 0 "J4" V 4975 6396 50  0000 C CNN
-F 1 "Conn_01x17" V 5066 6396 50  0000 C CNN
-F 2 "Connector_PinHeader_2.54mm:PinHeader_1x17_P2.54mm_Vertical" H 4850 6400 50  0001 C CNN
-F 3 "~" H 4850 6400 50  0001 C CNN
-	1    4850 6400
+P 4950 6400
+F 0 "J4" V 5075 6396 50  0000 C CNN
+F 1 "Conn_01x18" V 5166 6396 50  0000 C CNN
+F 2 "Connector_PinHeader_2.54mm:PinHeader_1x18_P2.54mm_Vertical" H 4950 6400 50  0001 C CNN
+F 3 "~" H 4950 6400 50  0001 C CNN
+	1    4950 6400
 	0    1    1    0
 $EndComp
@@
 Wire Wire Line
 	5750 5200 5750 4150
+$Comp
+L power:GND #PWR0101
+U 1 1 6032E2E7
+P 6000 6200
+F 0 "#PWR0101" H 6000 5950 50  0001 C CNN
+F 1 "GND" H 6005 6027 50  0000 C CNN
+F 2 "" H 6000 6200 50  0001 C CNN
+F 3 "" H 6000 6200 50  0001 C CNN
+	1    6000 6200
+	1    0    0    -1
+$EndComp
+Wire Wire Line
+	6000 6200 5750 6200
+$Comp
+L power:GND #PWR?
+U 1 1 60379D70
+P 3950 800
+F 0 "#PWR?" H 3950 550 50  0001 C CNN
+F 1 "GND" H 3955 627 50  0000 C CNN
+F 2 "" H 3950 800 50  0001 C CNN
+F 3 "" H 3950 800 50  0001 C CNN
+	1    3950 800
+	1    0    0    -1
+$EndComp
 $EndSCHEMATC
